File: KiCad/SimulateReceiver ESP32-S3-SuperMini/SimulateReceiver ESP32-S3-SuperMini.kicad_pcb (KiCad board)
At the start: 4 copper layers, 23.5 x 18 mm, 13 parts, among them IC1 CD4021BM96, J1 Conn_01x09, J2 Conn_01x09, J3 Conn_Coaxial, J4 Conn_01x06, U1 LM1881M, U2 ESP32-DevKitC

Commit message: Add files via upload
Other:
- board text added: "USB top"
- board text removed: "(USB top)"
Changed lines of the file:
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@@
 		(tags "connector Molex PicoBlade horizontal")
 		(property "Reference" "J4"
-			(at 3.176 1.572 270)
+			(at 0.4 1.75 270)
 			(layer "F.SilkS")
 			(effects
@@
 		)
 	)
-	(gr_text "(USB top)\n"
-		(at 101.75 95.75 90)
+	(gr_text "USB top\n"
+		(at 103.8 94.86 90)
 		(layer "F.SilkS")
 		(effects

Commit message: Add files via upload
Parts:
- J3: footprint Connector_PinHeader_2.54mm:PinHeader_1x02_P2.54mm_Vertical -> Connector_JST:JST_PH_S2B-PH-K_1x02_P2.00mm_Horizontal
- moved J3 2.57 mm to (122.3, 94.5), turned to 90 degrees
Routing:
- net Net-(J3-In): track 7.63 -> 7.12 mm

Commit message: Add files via upload
Parts:
- moved C2 0.92 mm to (123.9, 87.2)
- moved R1 0.82 mm to (121.5, 87.2)
- moved C1 0.37 mm to (118.8, 87.2)
- moved C4 0.21 mm to (116.3, 87.2)
Routing:
- net GND: track 6.23 -> 4.92 mm
- net Net-(U1-RSET): track 4.27 -> 4.84 mm

Commit message: Add files via upload
Parts:
- moved G*** 0.19 mm to (115.5, 85.9)
- turned C2 to 90 degrees
Routing:
- net Net-(U1-CVIN): track 9.88 -> 12.1 mm
- net Net-(J3-In): track 6.69 -> 5.43 mm, vias 1 -> 0
- net +5V: track 40.1 -> 40.9 mm
Other:
- board text added: "5V"
