File: KiCad/SimulateReceiver ESP32-S3-SuperMini/SimulateReceiver ESP32-S3-SuperMini.kicad_pcb (KiCad board)
At the start: 4 copper layers, 23.5 x 18 mm, 13 parts, among them IC1 CD4021BM96, J1 Conn_01x09, J2 Conn_01x09, J3 Conn_Coaxial, J4 Conn_01x06, U1 LM1881M, U2 ESP32-DevKitC

Commit message: Add files via upload
Routing:
- net +5V: track 41.0 -> 38.6 mm
Changed lines of the file:
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@@
 	)
 	(segment
-		(start 115.9 90.155)
-		(end 115.9 88.6775)
-		(width 0.5)
-		(layer "F.Cu")
-		(net 5)
-	)
-	(segment
-		(start 116.09 88.2775)
-		(end 115.1375 87.325)
-		(width 0.5)
-		(layer "F.Cu")
-		(net 5)
-	)
-	(segment
-		(start 115.9 91.367501)
+		(start 115.1375 87.325)
+		(end 113.8625 87.325)
+		(width 0.5)
+		(layer "F.Cu")
+		(net 5)
+	)
+	(segment
+		(start 112.755 88.595)
+		(end 113.825 88.595)
+		(width 0.5)
+		(layer "F.Cu")
+		(net 5)
+	)
+	(segment
+		(start 112.855 89.865)
+		(end 113.825 89.865)
+		(width 0.5)
+		(layer "F.Cu")
+		(net 5)
+	)
+	(segment
+		(start 112.675 87.325)
+		(end 113.825 87.325)
+		(width 0.5)
+		(layer "F.Cu")
+		(net 5)
+	)
+	(segment
+		(start 115.315 91.135)
 		(end 115.9 90.55)
 		(width 0.5)
@@
 	)
 	(segment
-		(start 115.425 91.842501)
-		(end 115.9 91.367501)
+		(start 112.49 88.86)
+		(end 112.755 88.595)
+		(width 0.5)
+		(layer "F.Cu")
+		(net 5)
+	)
+	(segment
+		(start 112.49 88.86)
+		(end 112.49 87.51)
 		(width 0.5)
 		(layer "F.Cu")
@@
 		(start 106.95 96.15)
 		(end 108.1 95)
+		(width 0.5)
+		(layer "F.Cu")
+		(net 5)
+	)
+	(segment
+		(start 112.85 89.86)
+		(end 112.855 89.865)
+		(width 0.5)
+		(layer "F.Cu")
+		(net 5)
+	)
+	(segment
+		(start 116.3 88.275)
+		(end 116.0875 88.275)
 		(width 0.5)
 		(layer "F.Cu")
@@
 	)
 	(segment
+		(start 112.49 90.22)
+		(end 112.85 89.86)
+		(width 0.5)
+		(layer "F.Cu")
+		(net 5)
+	)
+	(segment
+		(start 112.49 87.51)
+		(end 112.675 87.325)
+		(width 0.5)
+		(layer "F.Cu")
+		(net 5)
+	)
+	(segment
 		(start 106.95 96.15)
 		(end 105.85 96.15)
@@
 	)
 	(segment
-		(start 113.8625 89.865)
-		(end 115.61 89.865)
-		(width 0.5)
-		(layer "F.Cu")
-		(net 5)
-	)
-	(segment
-		(start 113.8625 88.595)
-		(end 116.1925 88.595)
-		(width 0.5)
-		(layer "F.Cu")
-		(net 5)
-	)
-	(segment
-		(start 115.9 88.6775)
-		(end 116.3 88.2775)
-		(width 0.5)
-		(layer "F.Cu")
-		(net 5)
-	)
-	(segment
-		(start 115.425 91.825)
-		(end 114.735 91.135)
+		(start 113.825 91.135)
+		(end 115.315 91.135)
+		(width 0.5)
+		(layer "F.Cu")
+		(net 5)
+	)
+	(segment
+		(start 113.8575 91.13)
+		(end 113.8625 91.135)
 		(width 0.5)
 		(layer "F.Cu")
@@
 	)
 	(segment
-		(start 115.425 91.842501)
-		(end 115.425 91.825)
-		(width 0.5)
-		(layer "F.Cu")
-		(net 5)
-	)
-	(segment
-		(start 114.735 91.135)
-		(end 113.8625 91.135)
-		(width 0.5)
-		(layer "F.Cu")
-		(net 5)
-	)
-	(segment
-		(start 115.1375 87.325)
-		(end 113.8625 87.325)
+		(start 116.0875 88.275)
+		(end 115.1375 87.325)
+		(width 0.5)
+		(layer "F.Cu")
+		(net 5)
+	)
+	(segment
+		(start 112.49 91.13)
+		(end 112.49 90.22)
+		(width 0.5)
+		(layer "F.Cu")
+		(net 5)
+	)
+	(segment
+		(start 112.49 90.22)
+		(end 112.49 88.86)
 		(width 0.5)
 		(layer "F.Cu")
@@
 	)
 	(segment
-		(start 115.61 89.865)
-		(end 115.9 90.155)
+		(start 112.49 91.13)
+		(end 113.8575 91.13)
 		(width 0.5)
 		(layer "F.Cu")
@@
 	)
 	(via blind
-		(at 115.425 91.842501)
+		(at 112.49 91.13)
 		(size 0.6)
 		(drill 0.3)
@@
 	)
 	(segment
-		(start 106.75 86.15)
-		(end 106.75 87.4)
-		(width 0.5)
+		(start 112.48 91.12)
+		(end 111.98 91.12)
+		(width 0.5)
+		(layer "B.Cu")
+		(net 5)
+	)
+	(segment
+		(start 104.8 85.8)
+		(end 106.4 85.8)
+		(width 0.5)
+		(layer "B.Cu")
+		(net 5)
+	)
+	(segment
+		(start 112.49 91.13)
+		(end 112.48 91.12)
+		(width 0.5)
+		(layer "B.Cu")
+		(net 5)
+	)
+	(segment
+		(start 111.98 91.12)
+		(end 106.95 96.15)
+		(width 0.5)
+		(layer "B.Cu")
+		(net 5)
+	)
+	(segment
+		(start 107.19 87.03)
+		(end 107.06 87.03)
+		(width 1)
 		(layer "B.Cu")
 		(net 5)
@@
 	)
 	(segment
-		(start 106.75 87.4)
-		(end 111.192501 91.842501)
-		(width 0.5)
-		(layer "B.Cu")
-		(net 5)
-	)
-	(segment
-		(start 111.257499 91.842501)
-		(end 115.425 91.842501)
-		(width 0.5)
-		(layer "B.Cu")
-		(net 5)
-	)
-	(segment
 		(start 106.4 85.8)
 		(end 106.75 86.15)
@@
 	)
 	(segment
-		(start 111.192501 91.842501)
-		(end 113 91.842501)
-		(width 0.5)
-		(layer "B.Cu")
-		(net 5)
-	)
-	(segment
-		(start 107.03 86.95)
-		(end 107.03 87.05)
-		(width 0.8)
-		(layer "B.Cu")
-		(net 5)
-	)
-	(segment
-		(start 106.95 96.15)
-		(end 111.257499 91.842501)
-		(width 0.5)
-		(layer "B.Cu")
-		(net 5)
-	)
-	(segment
-		(start 104.8 85.8)
-		(end 106.4 85.8)
+		(start 106.75 86.15)
+		(end 106.75 87.45)
+		(width 0.5)
+		(layer "B.Cu")
+		(net 5)
+	)
+	(segment
+		(start 106.75 87.45)
+		(end 111.2 91.9)
 		(width 0.5)
 		(layer "B.Cu")
@@
 	)
 	(segment
+		(start 118.425 94.075)
+		(end 117.17 95.33)
+		(width 0.2)
+		(layer "F.Cu")
+		(net 13)
+	)
+	(segment
 		(start 123.29 86.41)
 		(end 123.5 86.41)
 		(width 0.127)
-		(layer "F.Cu")
-		(net 13)
-	)
-	(segment
-		(start 118.5 94)
-		(end 117.17 95.33)
-		(width 0.2)
 		(layer "F.Cu")
 		(net 13)
@@
 	)
 	(via blind
-		(at 118.5 94)
+		(at 118.425 94.075)
 		(size 0.6)
 		(drill 0.3)
@@
 	)
 	(segment
+		(start 118.425 94.075)
+		(end 122.7 89.8)
+		(width 0.2)
+		(layer "B.Cu")
+		(net 13)
+	)
+	(segment
 		(start 122.7 89.8)
 		(end 122.7 89.7)
-		(width 0.2)
-		(layer "B.Cu")
-		(net 13)
-	)
-	(segment
-		(start 118.5 94)
-		(end 122.7 89.8)
 		(width 0.2)
 		(layer "B.Cu")
@@
 	)
 	(segment
-		(start 117.725 91.775)
-		(end 117.17 91.22)
+		(start 118.4 91.9)
+		(end 117.85 91.9)
 		(width 0.2)
 		(layer "F.Cu")
@@
 		(net 20)
 	)
+	(segment
+		(start 117.85 91.9)
+		(end 117.17 91.22)
+		(width 0.2)
+		(layer "F.Cu")
+		(net 20)
+	)
 	(via blind
-		(at 117.725 91.775)
+		(at 118.4 91.9)
 		(size 0.6)
 		(drill 0.3)
@@
 	)
 	(segment
-		(start 120.9 84.5)
-		(end 121.37728 84.02272)
+		(start 121.37728 84.02272)
+		(end 121.77728 84.02272)
 		(width 0.2)
 		(layer "B.Cu")
@@
 	)
 	(segment
-		(start 117.75 91.8)
-		(end 118.5 91.8)
-		(width 0.2)
-		(layer "B.Cu")
-		(net 20)
-	)
-	(segment
-		(start 121.37728 84.02272)
-		(end 121.77728 84.02272)
-		(width 0.2)
-		(layer "B.Cu")
-		(net 20)
-	)
-	(segment
-		(start 117.725 91.775)
-		(end 117.75 91.8)
-		(width 0.2)
-		(layer "B.Cu")
-		(net 20)
-	)
-	(segment
-		(start 118.5 91.8)
-		(end 120.9 89.4)
+		(start 120.9 84.5)
+		(end 121.37728 84.02272)
 		(width 0.2)
 		(layer "B.Cu")
@@
 		(layer "B.Cu")
 		(net 20)
+	)
+	(segment
+		(start 118.4 91.9)
+		(end 120.9 89.4)
+		(width 0.2)
+		(layer "B.Cu")
+		(net 20)
