File: KiCad/SimulateReceiver ESP32-S3-SuperMini/SimulateReceiver ESP32-S3-SuperMini.kicad_sch (KiCad schematic)
At the start: 12 parts, among them IC1 CD4021BM96, J1 Conn_01x09, J2 Conn_01x09, J3 Conn_Coaxial, J4 Conn_01x06, U1 LM1881M, U2 ESP32-DevKitC

Commit message: Add files via upload
Parts:
- J3: footprint Connector_PinHeader_2.54mm:PinHeader_1x02_P2.54mm_Vertical -> Connector_JST:JST_PH_S2B-PH-K_1x02_P2.00mm_Horizontal
Changed lines of the file:
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@@
 			)
 		)
-		(property "Footprint" "Connector_PinHeader_2.54mm:PinHeader_1x02_P2.54mm_Vertical"
+		(property "Footprint" "Connector_JST:JST_PH_S2B-PH-K_1x02_P2.00mm_Horizontal"
 			(at 44.45 96.52 0)
 			(effects

Commit message: Add files via upload
Changed lines of the file:
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@@
-	)
-	(no_connect
-		(at 34.29 63.5)
 	)
 	(no_connect
@@
 	)
 	(no_connect
+		(at 34.29 59.69)
+	)
+	(no_connect
 		(at 191.77 106.68)
 	)
@@
 		)
 		(stroke
+			(width 0)
+			(type default)
+		)
+	)
+	(wire
+		(pts
+			(xy 34.29 59.69) (xy 34.29 63.5)
+		)
+		(stroke
